File: KiCAD/PCB/YM60JIS_PCB .kicad_pcb (KiCad board)
At the start: 2 copper layers, 285.1 x 94.6 mm, 173 parts, among them J1 TYPE-C-31-M-12, SW1 SW_Push, SW10 SW_Push, SW11 SW_Push, SW12 SW_Push, SW13 SW_Push, SW14 SW_Push, SW15 SW_Push, SW16 SW_Push, SW17 SW_Push, SW18 SW_Push, SW19 SW_Push, SW2 SW_Push, SW20 SW_Push, SW21 SW_Push, SW22 SW_Push, SW23 SW_Push, SW24 SW_Push, SW25 SW_Push, SW26 SW_Push, SW27 SW_Push, SW28 SW_Push, SW29 Space, SW3 SW_Push, SW30 SW_Push, SW31 SW_Push, SW32 SW_Push, SW33 SW_Push, SW34 SW_Push, SW35 SW_Push, SW36 SW_Push, SW37 SW_Push, SW38 SW_Push, SW39 SW_Push, SW4 SW_Push, SW40 SW_Push, SW41 SW_Push, SW42 SW_Push, SW43 SW_Push, SW44 SW_Push, SW45 SW_Push, SW46 SW_Push, SW47 SW_Push, SW48 SW_Push, SW49 SW_Push, SW5 SW_Push, SW50 SW_Push, SW51 SW_Push, SW52 SW_Push, SW53 SW_Push, SW54 SW_Push, SW55 SW_Push, SW56 SW_Push, SW57 SW_Push, SW58 SW_Push, SW59 SW_Push, SW6 SW_Push, SW60 SW_Push, SW61 SW_Push, SW62 SW_Push, SW63 Yen, SW64 Backspace, SW65 ISOEnter, SW66 SW_Push, SW67 SW_Push, SW7 SW_Push, SW8 SW_Push, SW9 SW_Push, U1 XC6206P332MR, U2 SMF05CT1G, U3 RP2040, U4 W25Q16JVUXIQ, Y1 X322512MSB4SI

Commit message: PCBの設計データリネームとフォルダ移動
Parts:
- ?: renamed from REF**; value >VALUE -> (none)

Commit message: ライブラリの参照先をsubmodulesに変更
Parts:
- REF**: footprint Mounting_Keyboard_Stabilizer:Stabilizer_Cherry_MX_3.00u -> PCM_Mounting_Keyboard_Stabilizer:Stabilizer_Cherry_MX_3.00u
- SW1, SW11, SW12, SW13, SW14, SW16, SW17, SW18, SW19, SW21, SW22, SW23, SW24, SW25, SW26, SW27, SW28, SW30, SW31, SW32, SW33, SW34, SW35, SW36, SW37, SW38, SW39, SW40, SW41, SW43, SW44, SW45, SW46, SW48, SW49, SW50, SW51, SW53, SW54, SW55, SW56, SW57, SW58, SW59, SW6, SW60, SW61, SW62, SW63, SW64, SW66, SW67, SW7, SW8, SW9: footprint Switch_Keyboard_Hotswap_Kailh:SW_Hotswap_Kailh_MX_1.00u -> PCM_Switch_Keyboard_Hotswap_Kailh:SW_Hotswap_Kailh_MX_1.00u
- SW10, SW15, SW20, SW42, SW47, SW52: footprint Switch_Keyboard_Hotswap_Kailh:SW_Hotswap_Kailh_MX_1.25u -> PCM_Switch_Keyboard_Hotswap_Kailh:SW_Hotswap_Kailh_MX_1.25u
- SW2, SW5: footprint Switch_Keyboard_Hotswap_Kailh:SW_Hotswap_Kailh_MX_1.50u -> PCM_Switch_Keyboard_Hotswap_Kailh:SW_Hotswap_Kailh_MX_1.50u
- SW29: footprint Switch_Keyboard_Hotswap_Kailh:SW_Hotswap_Kailh_MX_3.00u -> PCM_Switch_Keyboard_Hotswap_Kailh:SW_Hotswap_Kailh_MX_3.00u
- SW3: footprint Switch_Keyboard_Hotswap_Kailh:SW_Hotswap_Kailh_MX_1.75u -> PCM_Switch_Keyboard_Hotswap_Kailh:SW_Hotswap_Kailh_MX_1.75u
- SW4: footprint Switch_Keyboard_Hotswap_Kailh:SW_Hotswap_Kailh_MX_2.00u -> PCM_Switch_Keyboard_Hotswap_Kailh:SW_Hotswap_Kailh_MX_2.00u
- SW65: footprint Switch_Keyboard_Hotswap_Kailh:SW_Hotswap_Kailh_MX_ISOEnter -> PCM_Switch_Keyboard_Hotswap_Kailh:SW_Hotswap_Kailh_MX_ISOEnter
- moved ? 0.50 mm to (120.5, 76.0)
Other:
- board text added: "."

Commit message: マウント穴の位置をGH60と同じ位置に調整
Parts:
- moved ? 0.69 mm to (355.6, 76.1)
- moved C9 0.65 mm to (124.0, 79.7), turned to -135 degrees
- moved ? 0.32 mm to (120.8, 76.1)
- moved C12 0.07 mm to (125.4, 77.7)
- moved C10 0.07 mm to (124.7, 78.4)
Routing:
- net GND: track 45.7 -> 46.9 mm
