File: KiCAD/PCB/YM60JIS_PCB.kicad_sch (KiCad schematic)
At the start: 165 parts, among them J1 TYPE-C-31-M-12, SW1 SW_Push, SW10 SW_Push, SW11 SW_Push, SW12 SW_Push, SW13 SW_Push, SW14 SW_Push, SW15 SW_Push, SW16 SW_Push, SW17 SW_Push, SW18 SW_Push, SW19 SW_Push, SW2 SW_Push, SW20 SW_Push, SW21 SW_Push, SW22 SW_Push, SW23 SW_Push, SW24 SW_Push, SW25 SW_Push, SW26 SW_Push, SW27 SW_Push, SW28 SW_Push, SW29 Space, SW3 SW_Push, SW30 SW_Push, SW31 SW_Push, SW32 SW_Push, SW33 SW_Push, SW34 SW_Push, SW35 SW_Push, SW36 SW_Push, SW37 SW_Push, SW38 SW_Push, SW39 SW_Push, SW4 SW_Push, SW40 SW_Push, SW41 SW_Push, SW42 SW_Push, SW43 SW_Push, SW44 SW_Push, SW45 SW_Push, SW46 SW_Push, SW47 SW_Push, SW48 SW_Push, SW49 SW_Push, SW5 SW_Push, SW50 SW_Push, SW51 SW_Push, SW52 SW_Push, SW53 SW_Push, SW54 SW_Push, SW55 SW_Push, SW56 SW_Push, SW57 SW_Push, SW58 SW_Push, SW59 SW_Push, SW6 SW_Push, SW60 SW_Push, SW61 SW_Push, SW62 SW_Push, SW63 Yen, SW64 Backspace, SW65 ISOEnter, SW66 SW_Push, SW67 SW_Push, SW7 SW_Push, SW8 SW_Push, SW9 SW_Push, U1 XC6206P332MR, U2 SMF05CT1G, U3 RP2040, U4 W25Q16JVUXIQ, Y1 X322512MSB4SI

Commit message: v1.1およびv1.1.1の追加
Parts:
- BTN1: JLCPCB Part # (none) -> C318884; LCSC Parts # C318884 -> (none)
- C1, C2: JLCPCB Part # (none) -> C15525; LCSC Parts # C15525 -> (none)
- C10, C13, C16, C17, C3, C4, C5, C6, C7, C8, C9: JLCPCB Part # (none) -> C1525; LCSC Parts # C1525 -> (none)
- C11, C12: JLCPCB Part # (none) -> C52923; LCSC Parts # C52923 -> (none)
- C14, C15: JLCPCB Part # (none) -> C1554; LCSC Parts # C1554 -> (none)
- D1, D10, D11, D12, D13, D14, D15, D16, D17, D18, D19, D2, D20, D21, D22, D23, D24, D25, D26, D27, D28, D29, D3, D30, D31, D32, D33, D34, D35, D36, D37, D38, D39, D4, D40, D41, D42, D43, D44, D45, D46, D47, D48, D49, D5, D50, D51, D52, D53, D54, D55, D56, D57, D58, D59, D6, D60, D61, D62, D63, D64, D65, D66, D67, D7, D8, D9: JLCPCB Part # (none) -> C81598; LCSC Parts # C81598 -> (none)
- J1: JLCPCB Part # (none) -> C165948; LCSC Parts # C165948 -> (none)
- R1, R3: JLCPCB Part # (none) -> C25905; LCSC Parts # C25905 -> (none)
- R4, R5: JLCPCB Part # (none) -> C13167; LCSC Parts # C13167 -> (none)
- R6, R8: JLCPCB Part # (none) -> C11702; LCSC Parts # C11702 -> (none)
- R7: JLCPCB Part # (none) -> C25744; LCSC Parts # C25744 -> (none)
- SW1, SW11, SW12, SW13, SW14, SW16, SW17, SW18, SW19, SW21, SW22, SW23, SW24, SW25, SW26, SW27, SW28, SW30, SW31, SW32, SW33, SW34, SW35, SW36, SW37, SW38, SW39, SW40, SW41, SW43, SW44, SW45, SW46, SW48, SW49, SW50, SW51, SW53, SW54, SW55, SW56, SW57, SW58, SW59, SW6, SW60, SW61, SW62, SW63, SW64, SW66, SW67, SW7, SW8, SW9: footprint PCM_Switch_Keyboard_Hotswap_Kailh:SW_Hotswap_Kailh_MX_1.00u -> PCM_marbastlib-mx:SW_MX_HS_CPG151101S11_1u; JLCPCB Part # (none) -> C41430893
- SW10, SW15, SW20, SW47, SW52: footprint PCM_Switch_Keyboard_Hotswap_Kailh:SW_Hotswap_Kailh_MX_1.25u -> PCM_marbastlib-mx:SW_MX_HS_CPG151101S11_1.25u; JLCPCB Part # (none) -> C41430893
- SW2, SW5: footprint PCM_Switch_Keyboard_Hotswap_Kailh:SW_Hotswap_Kailh_MX_1.50u -> PCM_marbastlib-mx:SW_MX_HS_CPG151101S11_1.5u; JLCPCB Part # (none) -> C41430893
- SW29: footprint PCM_Switch_Keyboard_Hotswap_Kailh:SW_Hotswap_Kailh_MX_3.00u -> PCM_marbastlib-mx:SW_MX_HS_CPG151101S11_1u; JLCPCB Part # (none) -> C41430893
- SW3: footprint PCM_Switch_Keyboard_Hotswap_Kailh:SW_Hotswap_Kailh_MX_1.75u -> PCM_marbastlib-mx:SW_MX_HS_CPG151101S11_1.75u; JLCPCB Part # (none) -> C41430893
- SW4: footprint PCM_Switch_Keyboard_Hotswap_Kailh:SW_Hotswap_Kailh_MX_2.00u -> PCM_marbastlib-mx:SW_MX_HS_CPG151101S11_1u; JLCPCB Part # (none) -> C41430893
- SW42: footprint PCM_Switch_Keyboard_Hotswap_Kailh:SW_Hotswap_Kailh_MX_1.25u -> PCM_marbastlib-mx:SW_MX_HS_CPG151101S11_1u; JLCPCB Part # (none) -> C41430893
- SW65: footprint PCM_Switch_Keyboard_Hotswap_Kailh:SW_Hotswap_Kailh_MX_ISOEnter -> PCM_marbastlib-mx:SW_MX_HS_CPG151101S11_1u; JLCPCB Part # (none) -> C41430893
- U1: JLCPCB Part # (none) -> C5446; LCSC Parts # C5446 -> (none)
- U2: JLCPCB Part # (none) -> C15879; LCSC Parts # C15879 -> (none)
- U3: JLCPCB Part # (none) -> C2040; LCSC Parts # C2040 -> (none)
- U4: JLCPCB Part # (none) -> C2843335; LCSC Parts # C2843335 -> (none)
- Y1: JLCPCB Part # (none) -> C9002; LCSC Parts # C9002 -> (none)

Commit message: 部品指定の誤りを修正
Parts:
- R4, R5: JLCPCB Part # C13167 -> C25190
Changed lines of the file:
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@@
 			)
 		)
-		(property "JLCPCB Part #" "C13167"
+		(property "JLCPCB Part #" "C25190"
 			(at 189.23 191.77 0)
 			(effects
@@
 			)
 		)
-		(property "JLCPCB Part #" "C13167"
+		(property "JLCPCB Part #" "C25190"
 			(at 182.88 189.23 0)
 			(effects
