File: KiCAD/Plate/YM60JIS_Plate.kicad_pcb (KiCad board)
At the start: 2 copper layers, 285.1 x 94.6 mm, 69 parts, among them SW1 SW_Push, SW10 SW_Push, SW11 SW_Push, SW12 SW_Push, SW13 SW_Push, SW14 SW_Push, SW15 SW_Push, SW16 SW_Push, SW17 SW_Push, SW18 SW_Push, SW19 SW_Push, SW2 SW_Push, SW20 SW_Push, SW21 SW_Push, SW22 SW_Push, SW23 SW_Push, SW24 SW_Push, SW25 SW_Push, SW26 SW_Push, SW27 SW_Push, SW28 SW_Push, SW29 Space, SW3 SW_Push, SW30 SW_Push, SW31 SW_Push, SW32 SW_Push, SW33 SW_Push, SW34 SW_Push, SW35 SW_Push, SW36 SW_Push, SW37 SW_Push, SW38 SW_Push, SW39 SW_Push, SW4 SW_Push, SW40 SW_Push, SW41 SW_Push, SW42 SW_Push, SW43 SW_Push, SW44 SW_Push, SW45 SW_Push, SW46 SW_Push, SW47 SW_Push, SW48 SW_Push, SW49 SW_Push, SW5 SW_Push, SW50 SW_Push, SW51 SW_Push, SW52 SW_Push, SW53 SW_Push, SW54 SW_Push, SW55 SW_Push, SW56 SW_Push, SW57 SW_Push, SW58 SW_Push, SW59 SW_Push, SW6 SW_Push, SW60 SW_Push, SW61 SW_Push, SW62 SW_Push, SW63 Yen, SW64 Backspace, SW65 ISOEnter, SW66 SW_Push, SW67 SW_Push, SW7 SW_Push, SW8 SW_Push, SW9 SW_Push

Commit message: PlateのライブラリパスをPCBと同様にsubmoduleへ変更、穴位置も微調整
Parts:
- moved ? 0.69 mm to (355.6, 76.1)
- moved REF** 0.67 mm to (120.8, 76.1)
Other:
- outline, holes or cut-outs redrawn
- board text added: "YM60JIS v1.0.1 @ymkn"
- board text removed: "YM60JIS v1.0 @ymkn"
Changed lines of the file:
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@@
   (title_block
     (title "YM60JIS Plate")
-    (date "2023-11-11")
-    (rev "v1.0")
+    (date "2024-01-08")
+    (rev "v1.0.1")
     (company "@ymkn")
   )
@@
     (pad_to_mask_clearance 0)
     (aux_axis_origin 95.25 47.625)
-    (grid_origin 95.25 47.625)
+    (grid_origin 95.55 48.225)
     (pcbplotparams
       (layerselection 0x00010fc_ffffffff)
@@
   )
   (footprint "kbd_Hole:m2_Spacer_Hole" locked (layer "F.Cu")
-    (at 120.45 75.525)
+    (at 120.75 76.125)
     (descr "Mounting Hole 2.2mm, no annular, M2")
     (tags "mounting hole 2.2mm no annular m2")
@@
   )
   (footprint "kbd_Hole:m2_Spacer_Hole" locked (layer "F.Cu")
-    (at 355.25 75.525)
+    (at 355.6 76.125)
     (descr "Mounting Hole 2.2mm, no annular, M2")
     (tags "mounting hole 2.2mm no annular m2")
@@
       (stroke (width 0.15) (type solid)) (layer "F.Fab"))
   )
-  (gr_line locked (start 380.6 140.825) (end 380.6 106.725)
+  (gr_line locked (start 380.6 140.825) (end 380.6 107.025)
     (stroke (width 0.1) (type default)) (layer "Edge.Cuts"))
-  (gr_arc locked (start 376.7 105.725) (mid 375.992894 105.432107) (end 375.7 104.725)
+  (gr_arc locked (start 376.7 106.025) (mid 375.992894 105.732107) (end 375.7 105.025)
     (stroke (width 0.1) (type default)) (layer "Edge.Cuts"))
   (gr_line locked (start 97.55 142.825) (end 378.6 142.825)
     (stroke (width 0.1) (type default)) (layer "Edge.Cuts"))
-  (gr_line locked (start 379.6 105.725) (end 376.7 105.725)
+  (gr_line locked (start 379.6 106.025) (end 376.7 106.025)
     (stroke (width 0.1) (type default)) (layer "Edge.Cuts"))
   (gr_arc locked (start 97.55 142.825) (mid 96.135786 142.239214) (end 95.55 140.825)
@@
   (gr_arc locked (start 95.55 50.225) (mid 96.135786 48.810786) (end 97.55 48.225)
     (stroke (width 0.1) (type default)) (layer "Edge.Cuts"))
-  (gr_arc locked (start 379.6 105.725) (mid 380.307106 106.017893) (end 380.6 106.725)
+  (gr_arc locked (start 379.6 106.025) (mid 380.307106 106.317893) (end 380.6 107.025)
     (stroke (width 0.1) (type default)) (layer "Edge.Cuts"))
-  (gr_arc (start 100.55 104.725) (mid 100.257107 105.432106) (end 99.55 105.725)
+  (gr_arc (start 100.55 105.025) (mid 100.257107 105.732106) (end 99.55 106.025)
     (stroke (width 0.1) (type default)) (layer "Edge.Cuts"))
-  (gr_line locked (start 380.6 102.225) (end 380.6 50.225)
+  (gr_line locked (start 380.6 101.925) (end 380.6 50.225)
     (stroke (width 0.1) (type default)) (layer "Edge.Cuts"))
   (gr_arc locked (start 378.6 48.225) (mid 380.014214 48.810786) (end 380.6 50.225)
     (stroke (width 0.1) (type default)) (layer "Edge.Cuts"))
-  (gr_arc locked (start 96.55 103.225) (mid 95.842894 102.932107) (end 95.55 102.225)
+  (gr_arc locked (start 96.55 102.925) (mid 95.842894 102.632107) (end 95.55 101.925)
     (stroke (width 0.1) (type default)) (layer "Edge.Cuts"))
-  (gr_line (start 95.55 106.727107) (end 95.55 140.825)
+  (gr_line (start 95.55 107.027107) (end 95.55 140.825)
     (stroke (width 0.1) (type default)) (layer "Edge.Cuts"))
-  (gr_line (start 100.55 104.725) (end 100.55 104.225)
+  (gr_line (start 100.55 105.025) (end 100.55 103.925)
     (stroke (width 0.1) (type default)) (layer "Edge.Cuts"))
-  (gr_line locked (start 96.55 103.225) (end 99.55 103.225)
+  (gr_line locked (start 96.55 102.925) (end 99.55 102.925)
     (stroke (width 0.1) (type default)) (layer "Edge.Cuts"))
-  (gr_line locked (start 375.7 104.225) (end 375.7 104.725)
+  (gr_line locked (start 375.7 103.925) (end 375.7 105.025)
     (stroke (width 0.1) (type default)) (layer "Edge.Cuts"))
-  (gr_arc locked (start 375.7 104.225) (mid 375.992893 103.517894) (end 376.7 103.225)
+  (gr_arc locked (start 375.7 103.925) (mid 375.992893 103.217894) (end 376.7 102.925)
     (stroke (width 0.1) (type default)) (layer "Edge.Cuts"))
-  (gr_line locked (start 95.55 50.225) (end 95.55 102.225)
+  (gr_line locked (start 95.55 50.225) (end 95.55 101.925)
     (stroke (width 0.1) (type default)) (layer "Edge.Cuts"))
-  (gr_arc (start 95.55 106.727107) (mid 95.843069 106.021024) (end 96.55 105.730004)
+  (gr_arc (start 95.55 107.027107) (mid 95.843067 106.321022) (end 96.55 106.030004)
     (stroke (width 0.1) (type default)) (layer "Edge.Cuts"))
-  (gr_arc locked (start 99.55 103.225) (mid 100.257106 103.517893) (end 100.55 104.225)
+  (gr_arc locked (start 99.55 102.925) (mid 100.257106 103.217893) (end 100.55 103.925)
     (stroke (width 0.1) (type default)) (layer "Edge.Cuts"))
-  (gr_line locked (start 379.6 103.225) (end 376.7 103.225)
+  (gr_line locked (start 379.6 102.925) (end 376.7 102.925)
     (stroke (width 0.1) (type default)) (layer "Edge.Cuts"))
   (gr_arc locked (start 380.6 140.825) (mid 380.014214 142.239214) (end 378.6 142.825)
     (stroke (width 0.1) (type default)) (layer "Edge.Cuts"))
-  (gr_arc locked (start 380.6 102.225) (mid 380.307107 102.932106) (end 379.6 103.225)
+  (gr_arc locked (start 380.6 101.925) (mid 380.307107 102.632106) (end 379.6 102.925)
     (stroke (width 0.1) (type default)) (layer "Edge.Cuts"))
   (gr_line locked (start 378.6 48.225) (end 97.55 48.225)
     (stroke (width 0.1) (type default)) (layer "Edge.Cuts"))
-  (gr_line locked (start 96.55 105.725) (end 99.55 105.725)
+  (gr_line locked (start 96.55 106.025) (end 99.55 106.025)
     (stroke (width 0.1) (type default)) (layer "Edge.Cuts"))
-  (gr_text "YM60JIS v1.0 @ymkn" (at 98.95 125.025 -270) (layer "B.SilkS")
+  (gr_text "YM60JIS v1.0.1 @ymkn" (at 98.95 125.025 90) (layer "B.SilkS")
     (effects (font (size 1 1) (thickness 0.15)) (justify left bottom mirror))
   )

Commit message: 左右のネジ穴を拡張、背面のテキストを除去
Other:
- outline, holes or cut-outs redrawn
- board text removed: "YM60JIS v1.0.1 @ymkn"
Changed lines of the file:
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@@
   (title_block
     (title "YM60JIS Plate")
-    (date "2024-01-08")
+    (date "2024-01-18")
     (rev "v1.0.1")
     (company "@ymkn")
@@
       (stroke (width 0.15) (type solid)) (layer "F.Fab"))
   )
-  (gr_line locked (start 380.6 140.825) (end 380.6 107.025)
+  (gr_line locked (start 380.6 140.825) (end 380.6 107.525)
     (stroke (width 0.1) (type default)) (layer "Edge.Cuts"))
-  (gr_arc locked (start 376.7 106.025) (mid 375.992894 105.732107) (end 375.7 105.025)
+  (gr_arc locked (start 376.7 106.525) (mid 375.992894 106.232107) (end 375.7 105.525)
     (stroke (width 0.1) (type default)) (layer "Edge.Cuts"))
   (gr_line locked (start 97.55 142.825) (end 378.6 142.825)
     (stroke (width 0.1) (type default)) (layer "Edge.Cuts"))
-  (gr_line locked (start 379.6 106.025) (end 376.7 106.025)
+  (gr_line locked (start 379.6 106.525) (end 376.7 106.525)
     (stroke (width 0.1) (type default)) (layer "Edge.Cuts"))
   (gr_arc locked (start 97.55 142.825) (mid 96.135786 142.239214) (end 95.55 140.825)
@@
   (gr_arc locked (start 95.55 50.225) (mid 96.135786 48.810786) (end 97.55 48.225)
     (stroke (width 0.1) (type default)) (layer "Edge.Cuts"))
-  (gr_arc locked (start 379.6 106.025) (mid 380.307106 106.317893) (end 380.6 107.025)
+  (gr_arc locked (start 379.6 106.525) (mid 380.307106 106.817893) (end 380.6 107.525)
     (stroke (width 0.1) (type default)) (layer "Edge.Cuts"))
-  (gr_arc (start 100.55 105.025) (mid 100.257107 105.732106) (end 99.55 106.025)
+  (gr_arc (start 100.55 105.525) (mid 100.257107 106.232106) (end 99.55 106.525)
     (stroke (width 0.1) (type default)) (layer "Edge.Cuts"))
-  (gr_line locked (start 380.6 101.925) (end 380.6 50.225)
+  (gr_line locked (start 380.6 101.425) (end 380.6 50.225)
     (stroke (width 0.1) (type default)) (layer "Edge.Cuts"))
   (gr_arc locked (start 378.6 48.225) (mid 380.014214 48.810786) (end 380.6 50.225)
     (stroke (width 0.1) (type default)) (layer "Edge.Cuts"))
-  (gr_arc locked (start 96.55 102.925) (mid 95.842894 102.632107) (end 95.55 101.925)
+  (gr_arc locked (start 96.55 102.425) (mid 95.842894 102.132107) (end 95.55 101.425)
     (stroke (width 0.1) (type default)) (layer "Edge.Cuts"))
-  (gr_line (start 95.55 107.027107) (end 95.55 140.825)
+  (gr_line (start 95.55 107.525) (end 95.55 140.825)
     (stroke (width 0.1) (type default)) (layer "Edge.Cuts"))
-  (gr_line (start 100.55 105.025) (end 100.55 103.925)
+  (gr_line (start 100.55 105.525) (end 100.55 103.425)
     (stroke (width 0.1) (type default)) (layer "Edge.Cuts"))
-  (gr_line locked (start 96.55 102.925) (end 99.55 102.925)
+  (gr_line locked (start 96.55 102.425) (end 99.55 102.425)
     (stroke (width 0.1) (type default)) (layer "Edge.Cuts"))
-  (gr_line locked (start 375.7 103.925) (end 375.7 105.025)
+  (gr_line locked (start 375.7 103.425) (end 375.7 105.525)
     (stroke (width 0.1) (type default)) (layer "Edge.Cuts"))
-  (gr_arc locked (start 375.7 103.925) (mid 375.992893 103.217894) (end 376.7 102.925)
+  (gr_arc locked (start 375.7 103.425) (mid 375.992893 102.717894) (end 376.7 102.425)
     (stroke (width 0.1) (type default)) (layer "Edge.Cuts"))
-  (gr_line locked (start 95.55 50.225) (end 95.55 101.925)
+  (gr_line locked (start 95.55 50.225) (end 95.55 101.425)
     (stroke (width 0.1) (type default)) (layer "Edge.Cuts"))
-  (gr_arc (start 95.55 107.027107) (mid 95.843067 106.321022) (end 96.55 106.030004)
+  (gr_arc (start 95.55 107.525) (mid 95.842466 106.817467) (end 96.55 106.525)
     (stroke (width 0.1) (type default)) (layer "Edge.Cuts"))
-  (gr_arc locked (start 99.55 102.925) (mid 100.257106 103.217893) (end 100.55 103.925)
+  (gr_arc locked (start 99.55 102.425) (mid 100.257106 102.717893) (end 100.55 103.425)
     (stroke (width 0.1) (type default)) (layer "Edge.Cuts"))
-  (gr_line locked (start 379.6 102.925) (end 376.7 102.925)
+  (gr_line locked (start 379.6 102.425) (end 376.7 102.425)
     (stroke (width 0.1) (type default)) (layer "Edge.Cuts"))
   (gr_arc locked (start 380.6 140.825) (mid 380.014214 142.239214) (end 378.6 142.825)
     (stroke (width 0.1) (type default)) (layer "Edge.Cuts"))
-  (gr_arc locked (start 380.6 101.925) (mid 380.307107 102.632106) (end 379.6 102.925)
+  (gr_arc locked (start 380.6 101.425) (mid 380.307107 102.132106) (end 379.6 102.425)
     (stroke (width 0.1) (type default)) (layer "Edge.Cuts"))
   (gr_line locked (start 378.6 48.225) (end 97.55 48.225)
     (stroke (width 0.1) (type default)) (layer "Edge.Cuts"))
-  (gr_line locked (start 96.55 106.025) (end 99.55 106.025)
+  (gr_line locked (start 96.55 106.525) (end 99.55 106.525)
     (stroke (width 0.1) (type default)) (layer "Edge.Cuts"))
-  (gr_text "YM60JIS v1.0.1 @ymkn" (at 98.95 125.025 90) (layer "B.SilkS")
-    (effects (font (size 1 1) (thickness 0.15)) (justify left bottom mirror))
-  )
 )
